Commit message: Fix inf ranges, update simuluation laserscan, reduce depth jump, add weight to wheels

File: gazebo/urdf/diff_bot.xacro (robot description, xacro)
@@ -36,6 +36,6 @@
         <friction>
           <ode>
-            <mu>0</mu>
-            <mu2>0</mu2>
+            <mu>0.0</mu>
+            <mu2>0.0</mu2>
             <slip1>1.0</slip1>
             <slip2>1.0</slip2>
@@ -50,5 +50,5 @@
       </geometry>
     </visual>
-    <collision name='caster_front_collision'>
+    <!--collision name='caster_front_collision'>
       <origin xyz="0.15 0 -0.05" rpy=" 0 0 0"/>
       <geometry>
@@ -71,5 +71,5 @@
         <sphere radius="0.05"/>
       </geometry>
-    </visual>
+    </visual-->
   </link>
   <link name="left_wheel">
@@ -89,5 +89,5 @@
     <inertial>
       <origin xyz="0 0 0" rpy="0 1.5707 1.5707"/>
-      <mass value="5"/>
+      <mass value="25"/>
       <inertia
         ixx=".1" ixy="0.0" ixz="0.0"
@@ -112,5 +112,5 @@
     <inertial>
       <origin xyz="0 0 0" rpy="0 1.5707 1.5707"/>
-      <mass value="5"/>
+      <mass value="25"/>
       <inertia
         ixx=".1" ixy="0.0" ixz="0.0"
@@ -126,5 +126,6 @@
     <axis xyz="0 1 0" rpy="0 0 0"/>
     <limit effort="10000" velocity="1000"/>
-    <joint_properties damping="1.0" friction="1.0"/>
+    <joint_properties damping="10.0" friction="0.0"/>
+    <!--joint_properties damping="1.0" friction="1.0"/-->
   </joint>
   <joint type="continuous" name="right_wheel_hinge">
@@ -135,5 +136,6 @@
     <axis xyz="0 1 0" rpy="0 0 0"/>
     <limit effort="10000" velocity="1000"/>
-    <joint_properties damping="1.0" friction="1.0"/>
+    <joint_properties damping="10.0" friction="0.0"/>
+    <!--joint_properties damping="1.0" friction="1.0"/-->
   </joint>
   <!--link name="camera">

Commit message: Change diff drive to 4 wheeled skid steer, change libgazebo_ros_diff_drive.so to libgazebo_ros_control.so

File: gazebo/urdf/diff_bot.xacro (robot description, xacro)
@@ -121,22 +121,42 @@
   <joint type="continuous" name="left_wheel_hinge">
     <origin xyz=".07 0.15 0" rpy="0 0 0"/>
-    <!--origin xyz="0.1 0.13 0" rpy="0 1.5707 1.5707"/-->
     <child link="left_wheel"/>
     <parent link="chassis"/>
     <axis xyz="0 1 0" rpy="0 0 0"/>
     <limit effort="10000" velocity="1000"/>
-    <joint_properties damping="10.0" friction="0.0"/>
-    <!--joint_properties damping="1.0" friction="1.0"/-->
+    <joint_properties damping="1.0" friction="1.0"/>
+    <implicitSpringDamper>1</implicitSpringDamper>
   </joint>
   <joint type="continuous" name="right_wheel_hinge">
     <origin xyz=".07 -0.15 0" rpy="0 0 0"/>
-    <!--origin xyz="0.1 -0.13 0" rpy="0 1.5707 1.5707"/-->
     <child link="right_wheel"/>
     <parent link="chassis"/>
     <axis xyz="0 1 0" rpy="0 0 0"/>
     <limit effort="10000" velocity="1000"/>
-    <joint_properties damping="10.0" friction="0.0"/>
-    <!--joint_properties damping="1.0" friction="1.0"/-->
+    <joint_properties damping="1.0" friction="1.0"/>
+    <implicitSpringDamper>1</implicitSpringDamper>
   </joint>
+  <transmission name="left_wheel_trans">
+    <type>transmission_interface/SimpleTransmission</type>
+    <joint name="left_wheel_hinge">
+      <hardwareInterface>hardware_interface/VelocityJointInterface</hardwareInterface>
+      <mechanicalReduction>1</mechanicalReduction>
+    </joint>
+    <actuator name="left_wheel_motor">
+      <mechanicalReduction>1</mechanicalReduction>
+      <hardwareInterface>VelocityJointInterface</hardwareInterface>
+    </actuator>
+  </transmission>
+  <transmission name="right_wheel_trans">
+    <type>transmission_interface/SimpleTransmission</type>
+    <joint name="right_wheel_hinge">
+      <hardwareInterface>hardware_interface/VelocityJointInterface</hardwareInterface>
+      <mechanicalReduction>1</mechanicalReduction>
+    </joint>
+    <actuator name="right_wheel_motor">
+      <mechanicalReduction>1</mechanicalReduction>
+      <hardwareInterface>VelocityJointInterface</hardwareInterface>
+    </actuator>
+  </transmission>
   <!--link name="camera">
     <collision>
@@ -192,3 +212,9 @@
     </inertial>
   </link>
+  <gazebo>
+    <plugin name="gazebo_ros_control" filename="libgazebo_ros_control.so">
+      <robotSimType>gazebo_ros_control/DefaultRobotHWSim</robotSimType>
+      <legacyModeNS>true</legacyModeNS>
+    </plugin>
+  </gazebo>
 </robot>
